File: test-project/test-project.kicad_pcb (KiCad board)
At the start: 2 copper layers, 75.5 x 38.1 mm, 24 parts, among them SW1 SW_Push, U1 ATmega32U4-A, Y1 16MHz

Commit message: roughly done with demo PCB
Routing:
- net unconnected-(USB1-SHIELD-Pad6): track 16.3 -> 0.00 mm
- added copper zone on B.Cu, net GND
Changed lines of the file:
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@@
     (property "ki_keywords" "diode")
     (attr smd)
-    (fp_text reference "D4" (at 0 2 90) (layer "B.SilkS")
+    (fp_text reference "D4" (at -3.89925 0 90) (layer "B.SilkS")
         (effects (font (size 1 1) (thickness 0.15)) (justify mirror))
     )
@@
         (effects (font (size 1 1) (thickness 0.15)) (justify mirror))
     )
-    (fp_text user "${REFERENCE}" (at 0 2 90) (layer "B.Fab")
+    (fp_text user "${REFERENCE}" (at -3.89925 0 90) (layer "B.Fab")
         (effects (font (size 1 1) (thickness 0.15)) (justify mirror))
     )
@@
         (effects (font (size 1 1) (thickness 0.15)) (justify mirror))
     )
-    (fp_text value "Molex-0548190589" (at -5.08 0) (layer "Dwgs.User")
+    (fp_text value "Molex-0548190589" (at -6.342 0) (layer "Dwgs.User") hide
         (effects (font (size 1 1) (thickness 0.15)))
     )
@@
     (property "ki_keywords" "switch normally-open pushbutton push-button")
     (attr smd)
-    (fp_text reference "SW1" (at 0 -4.064) (layer "B.SilkS")
+    (fp_text reference "SW1" (at 6.49275 -1.5855) (layer "B.SilkS")
         (effects (font (size 1 1) (thickness 0.15)) (justify mirror))
     )
@@
     (property "ki_keywords" "diode")
     (attr smd)
-    (fp_text reference "D2" (at 0 2 90) (layer "B.SilkS")
+    (fp_text reference "D2" (at -4.02825 0 90) (layer "B.SilkS")
         (effects (font (size 1 1) (thickness 0.15)) (justify mirror))
     )
@@
         (effects (font (size 1 1) (thickness 0.15)) (justify mirror))
     )
-    (fp_text user "${REFERENCE}" (at 0 2 90) (layer "B.Fab")
+    (fp_text user "${REFERENCE}" (at -4.02825 0 90) (layer "B.Fab")
         (effects (font (size 1 1) (thickness 0.15)) (justify mirror))
     )
@@
     (stroke (width 0.1) (type default)) (layer "Edge.Cuts"))
   (gr_arc (start 101.32125 77.6895) (mid 99.639573 76.992927) (end 98.943 75.31125)
+    (stroke (width 0.1) (type default)) (layer "Edge.Cuts"))
+  (gr_line (start 174.405 75.31125) (end 174.405 42.01575)
     (stroke (width 0.1) (type default)) (layer "Edge.Cuts"))
   (gr_arc (start 172.02675 39.6375) (mid 173.708427 40.334073) (end 174.405 42.01575)
@@
   (segment (start 117.969 46.6525) (end 116.942 47.6795) (width 0.254) (layer "B.Cu") (net 20))
   (segment (start 121.397303 52.661803) (end 121.90375 53.16825) (width 0.254) (layer "B.Cu") (net 20))
-  (segment (start 104.806 41.223) (end 104.806 45.723) (width 0.254) (layer "F.Cu") (net 44))
-  (segment (start 104.806 41.223) (end 112.106 41.223) (width 0.254) (layer "F.Cu") (net 44))
-  (segment (start 112.106 41.223) (end 112.106 45.723) (width 0.254) (layer "F.Cu") (net 44))
+  (zone (net 2) (net_name "GND") (layer "B.Cu") (hatch edge 0.5)
+    (connect_pads (clearance 0.5))
+    (min_thickness 0.25) (filled_areas_thickness no)
+    (fill yes (thermal_gap 0.5) (thermal_bridge_width 0.5))
+    (polygon
+      (pts
+        (xy 99.09375 39.6375)
+        (xy 136.353 39.6375)
+        (xy 136.353 77.6895)
+        (xy 99.09375 77.6895)
+      )
+    )
+  )
 )
